File: BriarPatch_Circuit/BriarPatch_Circuit.kicad_sch (KiCad schematic)
At the start: 12 parts, among them J1 LDR Module, J2 Solar Panel, U1 DFPlayer Mini, U2 RTC Module

Commit message: Updated circuit schematic to reflect addition of 15W speaker
Parts:
- removed BT1: 3.7V 3Ah Lipo, symbol Device:Battery_Cell
- removed CN3791: ~, symbol CN3791_SolarCharger:CN3791
- added C1, C2: 100uF, symbol Device:C
- added U3: PAM8610, symbol PAM8610:PAM8610
- added U4: LM2596S-5, Package_TO_SOT_SMD:TO-263-5_TabPin3, symbol Regulator_Switching:LM2596S-5
- J2: value Solar Panel -> 12V Power Supply
Connections:
- net +5V: now also C2.1, U4.2 (OUT); no longer A1.27 (+5V)
- net GND: now also J2.2 (Pin_2), C1.2, C2.2, U3. (Left-), U4.3 (GND)
- net +12V: now reaches J2.1 (Pin_1)
- net +12V: now also A1.30 (VIN), C1.1, U3. (Left-), U4.1 (VIN)
- net at U1.4 (DAC_R): now also U3. (Left-)
- net at U1.5 (DAC_L): now also U3. (Left-)
- net at LS1.1: now also U3. (Left-); no longer U1.6 (SPK1)
- net at LS1.2: now also U3. (Left-); no longer U1.8 (SPK2)
Other:
- moved on the sheet: R1, R2, U1
